File: TER kicad/TER kicad.kicad_sch (KiCad schematic)
At the start: 1 part

Commit message: Maj du kicad
Parts:
- added D1: LED, symbol Device:LED
- added DrMOS1: ~, symbol custom:Driver_Mosfet
- added Mot1: ~, symbol custom:BLDC
- added U1: 74AHC1G14, symbol 74xGxx:74AHC1G14
- added U2: CH340C, Package_SO:SOIC-16_3.9x9.9mm_P1.27mm, symbol Interface_USB:CH340C
Connections:
- net at CTRL1.10 (Vn): now also DrMOS1.5 (Vn)
- net at CTRL1.11 (Wn): now also DrMOS1.6 (Wn)
- net at CTRL1.12 (REV): now also D1.2 (A)
- net at CTRL1.4 (REV): now also U1.4
- net at CTRL1.6 (U): now also DrMOS1.1 (U)
- net at CTRL1.7 (V): now also DrMOS1.2 (V)
- net at CTRL1.8 (W): now also DrMOS1.3 (W)
- net at CTRL1.9 (Un): now also DrMOS1.4 (Un)
- new net: DrMOS1.7 (A), Mot1.1 (A)
- new net: DrMOS1.8 (B), Mot1.2 (B)
- new net: DrMOS1.9 (C), Mot1.3 (C)
- new net: Mot1.4 (Tour), U1.2
- new net GND: D1.1 (K), U1.3 (GND)
Other:
- moved on the sheet: CTRL1
