File: TER kicad/TER kicad.kicad_pcb (KiCad board)
At the start: 2 copper layers, 40.2 x 32 mm, 15 parts, among them J1 Conn_01x06_Pin, J2 Conn_01x02_Pin, U3 MOS

Commit message: Fix: nouveau branchement avec mosfet P
Other:
- board text removed: "SKIBIDILC"
Changed lines of the file:
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@@
-		)
-	)
-	(gr_text "SKIBIDILC"
-		(at 113.97 65.39 0)
-		(layer "F.SilkS")
-		(effects
-			(font
-				(size 1.2 1.2)
-				(thickness 0.3)
-				(bold yes)
-			)
-			(justify left bottom)
 		)
 	)
